File: Hardware/PCB/Blueberry Pi 7.1.2.esp32.no-lan.gsm-a9g.no-50p.sch (EAGLE design)
At the start: 231 parts, among them J2 AUDIO_JACK_SMD, J3 USB-A-FEMALE, Q1 24Mhz, Q2 32kHz, U1 MICROSIM, U2 W25Q32FV, U3 AP3031KTR-G1, U4 ESP-WROOM-32, U5 W25Q40BVSS, X1 FH12-50S-0.5SH, X2 53047-02

Commit message: better connected A9G module. added 'no-50pin lcd' schematic easier for router and with headers for the rest of A9G pins
Parts:
- removed C31, C6: 22uF/6.3V, rcl:C-EUC0805
- removed C32, C33, C35, C4, C40, C41, C42, C43: 100nF, rcl:C-EUC0603
- removed C5: 10uF/16V, rcl:C-EUC0805
- removed D3, D4: BAT54S, semicon-smd-ipc:DIODE_AC-AC_
- removed D5: 1N5819/SS14, gogo:SCHOTKKY7.62SSMINI-MELF
- removed JMP1, JMP2, JMP3: 0R-JUMPC, jump-0r-smd:0R-JUMPC
- removed L3: 47µH, induct-CD:INDUCTANCE_CD32
- removed R10, R7: 10k, rcl:R-EU_R0603
- removed R19, R40, R42: 51k/1%, rcl:R-EU_R0603_5MIL
- removed R34, R37, R41: 1k/1%, rcl:R-EU_R0603_5MIL
- removed R35: 20k, rcl:R-EU_R0603_5MIL
- removed R9: 30k, rcl:R-EU_R0603
- removed U3: AP3031KTR-G1, OLIMEX_IC:AP3031KTR-G1
- removed X1: FH12-50S-0.5SH, con-hirose:FH12-50S-0.5SH
- removed Z1: BZV55C6V8, gogo:ZDIOD-SMD
- removed Z2: BZV55C16, gogo:ZDIOD-SMD
- added DBG-COM1, DBG-COM2: HDR-1.27MM-110, headers-1.27:HDR-1.27MM-110
- added U$21: FH12-06S-0.5S, con-hirose:FH12-06S-0.5S
Connections:
- removed net -7V: C43.1, R41.1, R42.2, X1-42.1, Z1.A
- removed net 10.4V: C32.1, C5.1, D4.A, D5.C, R19.2, R35.2, U3.OV, X1-43.1
- removed net 16V: C40.1, R37.1, R40.2, R9.1, X1-41.1, Z2.C
- removed net L/R: JMP1-0R.2, X1-39.1
- removed net N$123: C33.1, C41.2, D5.A, L3.P$2, U3.SW
- removed net N$126: R19.1, R34.1, U3.FB
- removed net N$17: C4.1, R10.2, X1-44.1
- removed net N$24: JMP3-0R.2, X1-47.1
- removed net N$25: C33.2, D4.AK
- removed net N$27: C35.1, D4.K, R37.2
- removed net N$34: C42.1, D3.A, R41.2
- removed net N$37: C41.1, D3.AK
- removed net U/D: JMP2-0R.2, X1-40.1
- removed net VCOM: R7.1, R9.2, X1-46.1, X1-6.1
- new net A9G_HST_RXD: DBG-COM1.1, U6.HST_RXD
- new net A9G_HST_TXD: DBG-COM1.2, U6.HST_TXD
- new net A9G_IO26: DBG-COM2.7, U6.IO26
- new net A9G_IO27: DBG-COM2.8, U6.IO27
- new net A9G_IO28: DBG-COM2.9, U6.IO28
- new net A9G_IO29: DBG-COM1.8, U6.IO29
- new net A9G_IO30: DBG-COM2.10, U6.IO30
- new net A9G_LCD_CS: DBG-COM1.7, U6.LCD_CS
- new net A9G_LCD_DIO: DBG-COM1.5, U6.LCD_DIO
- new net A9G_LCD_RST: DBG-COM1.6, U6.LCD_RST
- new net A9G_LCD_SCK: DBG-COM1.3, U6.LCD_SCK
- new net A9G_LCD_SDC: DBG-COM1.4, U6.LCD_SDC
- new net A9G_SD_CLK: DBG-COM2.6, U6.SD_CLK
- new net A9G_SD_CMD: DBG-COM2.5, U6.SD_CMD
- new net A9G_SD_D0: DBG-COM2.4, U6.SD_D0
- new net A9G_SD_D1: DBG-COM2.3, U6.SD_D1
- new net A9G_SD_D2: DBG-COM2.2, U6.SD_D2
- new net A9G_SD_D3: DBG-COM2.1, U6.SD_D3
- new net N$85: J-LCD-FFC-1.MSV
- net !RESET: now also U$21.6
- net +3V3: now also DBG-COM1.9, U$21.5; no longer JMP1-0R.3, JMP2-0R.3, JMP3-0R.1, R10.1, X1-7.1, X1-8.1
- net +5V: no longer C31.2, C6.2, L3.P$1, U3.CTRL, U3.VIN
- net CSI_D0/LCD_D2: no longer X1-17.1
- net CSI_D1/LCD_D3: no longer X1-16.1
- net CSI_D10/LCD_D14: no longer X1-21.1
- net CSI_D11/LCD_D15: no longer X1-20.1
- net CSI_D12/LCD_D18: no longer X1-33.1
- net CSI_D2/LCD_D4: no longer X1-15.1
- net CSI_D3/LCD_D5: no longer X1-14.1
- net CSI_D4/LCD_D6: no longer X1-13.1
- net CSI_D5/LCD_D7: no longer X1-12.1
- net CSI_D6/LCD_D10: no longer X1-25.1
- net CSI_D7/LCD_D11: no longer X1-24.1
- net CSI_D8/LCD_D12: no longer X1-23.1
- net CSI_D9/LCD_D13: no longer X1-22.1
- net CSI_HSYNC/LCD_HSYNC: no longer X1-11.1
- net CSI_MCLK/LCD_DE: no longer X1-9.1
- net CSI_PCLK/LCD_CLK: no longer X1-37.1
- net CSI_VSYNC/LCD_VSYNC: no longer X1-10.1
- net GND: now also DBG-COM1.10, U$21.4; no longer C31.1, C32.2, C35.2, C4.2, C40.2, C42.2, C43.2, C5.2, C6.1, D3.K, JMP1-0R.1, JMP2-0R.1, JMP3-0R.3, R34.2, R35.1, R40.1, R42.1, R7.2, U3.GND, X1-18.1, X1-19.1, X1-26.1, X1-27.1, X1-34.1, X1-35.1, X1-36.1, X1-38.1, X1-48.1, X1-5.1, Z1.C, Z2.A
- net HP_L: no longer J-AUDIO.3
- net HP_L_O: now also J-AUDIO.3
- net HP_R: no longer J-AUDIO.2
- net HP_R_O: now also J-AUDIO.2
- net I2C1/SCL: now also U$21.1
- net I2C1/SDA: now also U$21.2
- net LCD_D19: no longer X1-32.1
- net LCD_D20: no longer X1-31.1
- net LCD_D21: no longer X1-30.1
- net LCD_D22: no longer X1-29.1
- net LCD_D23: no longer X1-28.1
- net PB3: now also U$21.3
- net VLED+: no longer X1-1.1, X1-2.1
- net VLED-: no longer J-LCD-FFC-1.MSV, X1-3.1, X1-4.1
Other:
- note removed: "2.7-16V"
- note removed: "Ra"
- note removed: "Rb"
- note removed: "Vout=0.2*(1+Ra/Rb)=10.4V"
